File: kicad-projects/old-ram-slice/ram-slice/ram-slice.sch (KiCad schematic (older format))
At the start: 27 parts, among them J1 Conn_02x24_Counter_Clockwise, J2 Conn_02x24_Counter_Clockwise, Q1 BS170, Q10 BS170, Q11 BS170, Q12 BS170, Q13 BS170, Q2 BS170, Q3 BS170, Q4 BS170, Q5 BS170, Q6 BS170, Q7 BS170, Q8 BS170, Q9 BS170, U1 IS61C5128AS-25QLI, U10 74LS08, U12 27C64, U15 74LS02, U17 74LS32, U2 IS61C5128AS-25QLI, U3 74LS04, U4 74LS08, U5 74LS10, U6 74LS10, U7 74LS00, U9 27C64

Commit message: stuff
Connections:
- net GND: now reaches U10.7 (GND)
- net GND: now also U15.7 (GND), U17.7 (GND), U3.7 (GND), U5.7 (GND), U6.7 (GND), U7.7 (GND)
- net VCC: now reaches U15.14 (VCC)
- net VCC: now also U17.14 (VCC), U3.14 (VCC), U5.14 (VCC), U6.14 (VCC), U7.14 (VCC)
Changed lines of the file:
@@
 Text Label 15600 3350 2    50   ~ 0
 ~HIGH_RAM_ENABLE
+$Comp
+L power:VCC #PWR?
+U 1 1 5F25B78C
+P 6650 8900
+F 0 "#PWR?" H 6650 8750 50  0001 C CNN
+F 1 "VCC" H 6665 9073 50  0000 C CNN
+F 2 "" H 6650 8900 50  0001 C CNN
+F 3 "" H 6650 8900 50  0001 C CNN
+	1    6650 8900
+	1    0    0    -1
+$EndComp
+$Comp
+L power:VCC #PWR?
+U 1 1 5F25C330
+P 7650 8850
+F 0 "#PWR?" H 7650 8700 50  0001 C CNN
+F 1 "VCC" H 7665 9023 50  0000 C CNN
+F 2 "" H 7650 8850 50  0001 C CNN
+F 3 "" H 7650 8850 50  0001 C CNN
+	1    7650 8850
+	1    0    0    -1
+$EndComp
+$Comp
+L power:GND #PWR?
+U 1 1 5F25DC47
+P 6650 9900
+F 0 "#PWR?" H 6650 9650 50  0001 C CNN
+F 1 "GND" H 6655 9727 50  0000 C CNN
+F 2 "" H 6650 9900 50  0001 C CNN
+F 3 "" H 6650 9900 50  0001 C CNN
+	1    6650 9900
+	1    0    0    -1
+$EndComp
+$Comp
+L power:GND #PWR?
+U 1 1 5F2606D9
+P 7650 9850
+F 0 "#PWR?" H 7650 9600 50  0001 C CNN
+F 1 "GND" H 7655 9677 50  0000 C CNN
+F 2 "" H 7650 9850 50  0001 C CNN
+F 3 "" H 7650 9850 50  0001 C CNN
+	1    7650 9850
+	1    0    0    -1
+$EndComp
+$Comp
+L power:GND #PWR?
+U 1 1 5F261F54
+P 3650 11900
+F 0 "#PWR?" H 3650 11650 50  0001 C CNN
+F 1 "GND" H 3655 11727 50  0000 C CNN
+F 2 "" H 3650 11900 50  0001 C CNN
+F 3 "" H 3650 11900 50  0001 C CNN
+	1    3650 11900
+	1    0    0    -1
+$EndComp
+$Comp
+L power:GND #PWR?
+U 1 1 5F263306
+P 12000 10500
+F 0 "#PWR?" H 12000 10250 50  0001 C CNN
+F 1 "GND" H 12005 10327 50  0000 C CNN
+F 2 "" H 12000 10500 50  0001 C CNN
+F 3 "" H 12000 10500 50  0001 C CNN
+	1    12000 10500
+	1    0    0    -1
+$EndComp
+$Comp
+L power:GND #PWR?
+U 1 1 5F26470B
+P 13950 14550
+F 0 "#PWR?" H 13950 14300 50  0001 C CNN
+F 1 "GND" H 13955 14377 50  0000 C CNN
+F 2 "" H 13950 14550 50  0001 C CNN
+F 3 "" H 13950 14550 50  0001 C CNN
+	1    13950 14550
+	1    0    0    -1
+$EndComp
+$Comp
+L power:GND #PWR?
+U 1 1 5F266E95
+P 18400 14600
+F 0 "#PWR?" H 18400 14350 50  0001 C CNN
+F 1 "GND" H 18405 14427 50  0000 C CNN
+F 2 "" H 18400 14600 50  0001 C CNN
+F 3 "" H 18400 14600 50  0001 C CNN
+	1    18400 14600
+	1    0    0    -1
+$EndComp
+$Comp
+L power:GND #PWR?
+U 1 1 5F2682B2
+P 20500 14400
+F 0 "#PWR?" H 20500 14150 50  0001 C CNN
+F 1 "GND" H 20505 14227 50  0000 C CNN
+F 2 "" H 20500 14400 50  0001 C CNN
+F 3 "" H 20500 14400 50  0001 C CNN
+	1    20500 14400
+	1    0    0    -1
+$EndComp
+$Comp
+L power:VCC #PWR?
+U 1 1 5F269BF0
+P 12000 9500
+F 0 "#PWR?" H 12000 9350 50  0001 C CNN
+F 1 "VCC" H 12015 9673 50  0000 C CNN
+F 2 "" H 12000 9500 50  0001 C CNN
+F 3 "" H 12000 9500 50  0001 C CNN
+	1    12000 9500
+	1    0    0    -1
+$EndComp
+$Comp
+L power:VCC #PWR?
+U 1 1 5F26B7B5
+P 18400 13600
+F 0 "#PWR?" H 18400 13450 50  0001 C CNN
+F 1 "VCC" H 18415 13773 50  0000 C CNN
+F 2 "" H 18400 13600 50  0001 C CNN
+F 3 "" H 18400 13600 50  0001 C CNN
+	1    18400 13600
+	1    0    0    -1
+$EndComp
+$Comp
+L power:VCC #PWR?
+U 1 1 5F26CC0B
+P 20500 13400
+F 0 "#PWR?" H 20500 13250 50  0001 C CNN
+F 1 "VCC" H 20515 13573 50  0000 C CNN
+F 2 "" H 20500 13400 50  0001 C CNN
+F 3 "" H 20500 13400 50  0001 C CNN
+	1    20500 13400
+	1    0    0    -1
+$EndComp
+$Comp
+L power:VCC #PWR?
+U 1 1 5F26E9B4
+P 3650 10900
+F 0 "#PWR?" H 3650 10750 50  0001 C CNN
+F 1 "VCC" H 3665 11073 50  0000 C CNN
+F 2 "" H 3650 10900 50  0001 C CNN
+F 3 "" H 3650 10900 50  0001 C CNN
+	1    3650 10900
+	1    0    0    -1
+$EndComp
 $EndSCHEMATC
