File: kicad-projects/mmio-unit/mmio-unit.sch (KiCad schematic (older format))
At the start: 29 parts, among them U1 4072, U10 74LS10, U11 74LS20, U12 74HC245, U13 74HC245, U14 74HC244, U15 74HC244, U2 4072, U3 IS61C5128AS-25QLI, U4 AT28C64B-15PU, U5 74LS02, U6 74LS08, U7 IS61C5128AS-25QLI, U8 AT28C64B-15PU, U9 74LS10

Commit message: vmem
Parts:
- removed unit 1 of U1
- removed unit 2 of U1
- removed unit 1 of U2
- removed unit 2 of U2
- added D1, D10, D11, D2, D3, D4, D5, D6, D7, D8, D9: 1N4148W, Diode_SMD:D_SOD-123, symbol Diode:1N4148W
- added R1: 10k, symbol Device:R
- gave numbers to parts that had none: 7
Connections:
- net D0: now also U18.3 (D0)
- net D1: now also U18.4 (D1)
- net D2: now also U18.7 (D2)
- net D3: now also U18.8 (D3)
- net D4: now also U18.13 (D4)
- net D5: now also U18.14 (D5)
- net D6: now also U18.17 (D6)
- net D7: now also U18.18 (D7)
- net GND: now also U18.10 (GND), R1.1
- net PA10: now also D2.2 (A)
- net PA11: now also D3.2 (A)
- net PA12: now also D4.2 (A)
- net PA13: now also D5.2 (A)
- net PA14: now also D6.2 (A)
- net PA15: now also D7.2 (A)
- net PA16: now also D8.2 (A)
- net PA17: now also D9.2 (A)
- net PA18: now also D10.2 (A)
- net PA19: now also D11.2 (A)
- net PA9: now also D1.2 (A)
- net VCC: now also U18.20 (VCC)
- net at U6.1: now also D1.1 (K), D10.1 (K), D11.1 (K), D2.1 (K), D3.1 (K), D4.1 (K), D5.1 (K), D6.1 (K), D7.1 (K), D8.1 (K), D9.1 (K), R1.2
- net PTB4: now reaches U18.12 (O4)
- net PTB5: now reaches U18.15 (O5)
- net PTB6: now reaches U18.16 (O6)
- net PTB7: now reaches U18.19 (O7)
- net PTB0: now reaches U18.2 (O0)
- net PTB1: now reaches U18.5 (O1)
- net PTB2: now reaches U18.6 (O2)
- net PTB3: now reaches U18.9 (O3)
Other:
- moved on the sheet: U5A, U5B, U6A
